Commit message: URDF for MiR250

File: mir_description/urdf/include/common.gazebo.xacro (robot description, xacro)
@@ -3,10 +3,11 @@
   <xacro:macro name="controller_plugin_gazebo" params="robot_namespace">
     <gazebo>
-      <plugin name="gazebo_ros_control" filename="libgazebo_ros_control.so">
+      <plugin filename="libgazebo_ros2_control.so" name="gazebo_ros2_control">
+        <robot_param>robot_description</robot_param>
+        <robot_param_node>robot_state_publisher</robot_param_node>
         <xacro:unless value="${robot_namespace == ''}">
-          <robotNamespace>${robot_namespace}</robotNamespace>
+          <robot_namespace>${robot_namespace}</robot_namespace>
         </xacro:unless>
-        <controlPeriod>0.001</controlPeriod>
-        <legacyModeNS>false</legacyModeNS>
+        <control_period>0.001</control_period>
       </plugin>
     </gazebo>

File: mir_description/urdf/include/common_properties.urdf.xacro (robot description, xacro)
@@ -50,4 +50,9 @@
     </material>
   </xacro:property>
+  <xacro:property name="material_red">
+    <material name="red">
+      <color rgba="1 0 0 1" />
+    </material>
+  </xacro:property>
   <!-- #################### inertials with origin #################### -->
   <!-- see https://secure.wikimedia.org/wikipedia/en/wiki/List_of_moment_of_inertia_tensors -->

File: mir_description/urdf/include/imu.gazebo.urdf.xacro (robot description, xacro)
@@ -10,18 +10,74 @@
       <xacro:property name="imu_frame" value="$(arg tf_prefix)/imu_frame" />
   </xacro:unless>
-  <xacro:macro name="imu_gazebo" params="link imu_topic update_rate">
-    <gazebo>
-      <plugin name="imu_plugin" filename="libhector_gazebo_ros_imu.so">
-        <updateRate>${update_rate}</updateRate>
-        <bodyName>${link}</bodyName>
-        <frameId>${imu_frame}</frameId>  <!-- from real MiR -->
-        <topicName>${imu_topic}</topicName>
-        <accelDrift>0.0 0.0 0.0</accelDrift>
-        <accelGaussianNoise>${sqrt(5e-05)} ${sqrt(0.0001)} ${sqrt(0.00013)}</accelGaussianNoise>    <!-- real MiR linear_acceleration_covariance: [5e-05, 0.0, 0.0, 0.0, 0.0001, 0.0, 0.0, 0.0, 0.00013] -->
-        <rateDrift>0.0 0.0 0.0</rateDrift>
-        <rateGaussianNoise>${sqrt(8e-06)} ${sqrt(8e-06)} ${sqrt(3e-07)}</rateGaussianNoise>         <!-- real MiR angular_velocity_covariance: [8e-06, 0.0, 0.0, 0.0, 8e-06, 0.0, 0.0, 0.0, 3e-07] -->
-        <yawDrift>0.0</yawDrift>
-        <yawGaussianNoise>${sqrt(0.1)}</yawGaussianNoise>                                           <!-- real MiR orientation_covariance: [0.1, 0.0, 0.0, 0.0, 0.1, 0.0, 0.0, 0.0, 0.1] -->
-      </plugin>
+  <xacro:macro name="imu_gazebo" params="link imu_topic update_rate stdev">
+    <gazebo reference="${link}">
+      <gravity>true</gravity>
+      <sensor name="imu_sensor" type="imu">
+        <always_on>true</always_on>
+        <update_rate>${update_rate}</update_rate>
+        <visualize>true</visualize>
+        <imu>
+          <angular_velocity>
+            <x>
+              <noise type="gaussian">
+                <mean>0.0</mean>
+                <stddev>${stdev}</stddev>
+                <bias_mean>0.0000075</bias_mean>
+                <bias_stddev>0.0000008</bias_stddev>
+              </noise>
+            </x>
+            <y>
+              <noise type="gaussian">
+                <mean>0.0</mean>
+                <stddev>${stdev}</stddev>
+                <bias_mean>0.0000075</bias_mean>
+                <bias_stddev>0.0000008</bias_stddev>
+              </noise>
+            </y>
+            <z>
+              <noise type="gaussian">
+                <mean>0.0</mean>
+                <stddev>${stdev}</stddev>
+                <bias_mean>0.0000075</bias_mean>
+                <bias_stddev>0.0000008</bias_stddev>
+              </noise>
+            </z>
+          </angular_velocity>
+          <linear_acceleration>
+            <x>
+              <noise type="gaussian">
+                <mean>0.0</mean>
+                <stddev>${stdev}</stddev>
+                <bias_mean>0.1</bias_mean>
+                <bias_stddev>0.001</bias_stddev>
+              </noise>
+            </x>
+            <y>
+              <noise type="gaussian">
+                <mean>0.0</mean>
+                <stddev>${stdev}</stddev>
+                <bias_mean>0.1</bias_mean>
+                <bias_stddev>0.001</bias_stddev>
+              </noise>
+            </y>
+            <z>
+              <noise type="gaussian">
+                <mean>0.0</mean>
+                <stddev>${stdev}</stddev>
+                <bias_mean>0.1</bias_mean>
+                <bias_stddev>0.001</bias_stddev>
+              </noise>
+            </z>
+          </linear_acceleration>
+        </imu>
+        <plugin filename="libgazebo_ros_imu_sensor.so" name="imu_plugin">
+        <initial_orientation_as_reference>false</initial_orientation_as_reference>
+          <ros>
+            <namespace>${imu_topic}</namespace>
+            <remapping>~/out:=data</remapping>
+            <frame_name>${imu_frame}</frame_name>  <!-- from real MiR -->
+          </ros>
+        </plugin>
+      </sensor>
     </gazebo>
   </xacro:macro>

File: mir_description/urdf/include/mir_100_v1.urdf.xacro (robot description, xacro)
@@ -1,9 +1,151 @@
 <?xml version="1.0"?>
-<robot xmlns:xacro="http://ros.org/wiki/xacro"
-       name="mir_100" >
-  <!-- This file is only for backward compatibility before the "mir_100" to "mir" rename. -->
-  <xacro:include filename="$(find mir_description)/urdf/include/mir_v1.urdf.xacro" />
-  <xacro:macro name="mir_100" params="prefix">
-    <xacro:mir prefix="${prefix}" />
+<robot xmlns:xacro="http://ros.org/wiki/xacro">
+  <xacro:include filename="$(find mir_description)/urdf/include/common_properties.urdf.xacro" />
+  <xacro:include filename="$(find mir_description)/urdf/include/imu.gazebo.urdf.xacro" />
+  <xacro:include filename="$(find mir_description)/urdf/include/mir_100.gazebo.xacro" />
+  <xacro:include filename="$(find mir_description)/urdf/include/mir_100.transmission.xacro" />
+  <xacro:include filename="$(find mir_description)/urdf/include/sick_s300.urdf.xacro" />
+  <xacro:include filename="$(find mir_description)/urdf/include/wheel.urdf.xacro" />
+  <xacro:include filename="$(find mir_description)/urdf/include/caster.urdf.xacro" />
+  <xacro:property name="deg_to_rad" value="0.017453293" />
+  <!-- The inertia for the MiR platform is intentionally chosen to be smaller than
+       the bounding box and also shifted a bit to the back, because most of the mass
+       is in the lower center back (because of the batteries). -->
+  <xacro:property name="mir_base_inertial_x" value="-0.05" />
+  <xacro:property name="mir_base_inertial_y" value="0.0" />
+  <xacro:property name="mir_base_inertial_z" value="0.15" />
+  <xacro:property name="mir_base_inertial_x_length" value="0.50" />
+  <xacro:property name="mir_base_inertial_y_length" value="0.30" />
+  <xacro:property name="mir_base_inertial_z_length" value="0.20" />
+  <xacro:property name="mir_100_act_wheel_radius" value="0.100" />
+  <xacro:property name="mir_100_act_wheel_width" value="0.038" />
+  <xacro:property name="mir_100_act_wheel_mass" value="1.0" />
+  <!--xacro:property name="mir_100_act_wheel_dx" value="0.037646" /-->
+  <xacro:property name="mir_100_act_wheel_dx" value="-0.004485" />
+  <!--xacro:property name="mir_100_act_wheel_dy" value="0.222604" /-->
+  <xacro:property name="mir_100_act_wheel_dy" value="0.2015" />
+  <xacro:property name="mir_100_caster_wheel_radius" value="0.0625" />
+  <xacro:property name="mir_100_caster_wheel_width" value="0.032" />
+  <xacro:property name="mir_100_caster_wheel_mass" value="1.0" />
+  <xacro:property name="mir_100_caster_wheel_dx" value="-0.0382" />
+  <xacro:property name="mir_100_caster_wheel_dy" value="0" />
+  <xacro:property name="mir_100_caster_wheel_dz" value="-0.094" />
+  <!--xacro:property name="mir_100_front_caster_wheel_base_dx" value="0.341346" /-->
+  <xacro:property name="mir_100_front_caster_wheel_base_dx" value="0.3037" />
+  <!--xacro:property name="mir_100_back_caster_wheel_base_dx" value="-0.270154" /-->
+  <xacro:property name="mir_100_back_caster_wheel_base_dx" value="-0.296" />
+  <!--xacro:property name="mir_100_caster_wheel_base_dy" value="0.203" /-->
+  <xacro:property name="mir_100_caster_wheel_base_dy" value="0.188" />
+  <xacro:property name="mir_100_caster_wheel_base_dz" value="${mir_100_caster_wheel_radius - mir_100_caster_wheel_dz}" />
+  <!-- MiR 100 complete mass 78.2kg (8.2kg battery) -->
+  <!-- - 2x2kg sick laser = 4kg-->
+  <!-- - 4x caster wheels + rotation link: 4x 1.31 kg -->
+  <!-- - 2x act wheels: 2kg -->
+  <!--xacro:property name="mir_100_base_mass" value="66.96" /-->
+  <xacro:property name="mir_100_base_mass" value="97.0" />
+  <xacro:property name="imu_stdev" value="0.00017" />
+  <xacro:macro name="mir_100" params="prefix ns">
+    <link name="${prefix}base_footprint" />
+    <joint name="${prefix}base_joint" type="fixed">
+      <parent link="${prefix}base_footprint" />
+      <child link="${prefix}base_link" />
+      <origin xyz="0 0 0" rpy="0 0 0" />
+    </joint>
+    <link name="${prefix}base_link">
+      <xacro:box_inertial mass="${mir_100_base_mass}" x="${mir_base_inertial_x_length}" y="${mir_base_inertial_y_length}" z="${mir_base_inertial_z_length}">
+        <origin xyz="${mir_base_inertial_x + mir_100_act_wheel_dx} ${mir_base_inertial_y} ${mir_base_inertial_z}" rpy="0 0 0" />
+      </xacro:box_inertial>
+      <visual>
+        <origin xyz="${mir_100_act_wheel_dx} 0 0" rpy="0 0 0" />
+        <geometry>
+          <!--mesh filename="package://mir_description/meshes/visual/mir_100_base.stl" /-->
+          <mesh filename="package://mir_description/meshes/visual/mir_250_base.stl" />
+        </geometry>
+        <!--xacro:insert_block name="material_white" /-->
+        <xacro:insert_block name="material_light_grey" />
+      </visual>
+      <collision>
+        <origin xyz="${mir_100_act_wheel_dx} 0 0" rpy="0 0 0" />
+        <geometry>
+          <!--mesh filename="package://mir_description/meshes/collision/mir_100_base.stl" /-->
+          <mesh filename="package://mir_description/meshes/collision/mir_250_base.stl" />
+        </geometry>
+      </collision>
+    </link>
+    <gazebo reference="${prefix}base_link">
+      <!--material>Gazebo/White</material-->
+      <material>Gazebo/Grey</material>
+    </gazebo>
+    <!-- IMU -->
+    <joint name="${prefix}base_link_to_imu_joint" type="fixed">
+      <parent link="${prefix}base_link" />
+      <child link="${prefix}imu_link" />
+      <origin xyz="0.0 0.0 0.25" rpy="0 0 0" />  <!-- same as real MiR -->
+    </joint>
+    <link name="${prefix}imu_link" />
+    <xacro:imu_gazebo link="${prefix}imu_link" imu_topic="${prefix}imu_data" update_rate="50.0" stdev="${imu_stdev}" />
+    <!-- Create an alias for imu_link. This is necessary because the real MiR's
+         TF has imu_link, but the imu_data topic is published in the imu_frame
+         frame. -->
+    <joint name="${prefix}imu_link_to_imu_frame_joint" type="fixed">
+      <parent link="${prefix}imu_link" />
+      <child link="${prefix}imu_frame" />
+      <origin xyz="0 0 0" rpy="0 0 0" />
+    </joint>
+    <link name="${prefix}imu_frame" />
+    <!-- Laser scanners -->
+    <!-- virtual link for merged laserscan-->
+    <joint name="${prefix}base_link_to_virtual_laser_joint" type="fixed">
+      <parent link="${prefix}base_link" />
+      <child link="${prefix}virtual_laser_link" />
+      <origin xyz="0.0 0.0 0.25" rpy="0.0 0.0 0" />
+    </joint>
+    <link name="${prefix}virtual_laser_link">
+    </link>
+    <joint name="${prefix}base_link_to_front_laser_joint" type="fixed">
+      <parent link="${prefix}base_link" />
+      <child link="${prefix}front_laser_link" />
+      <!--origin xyz="0.3564 0.2064 0.1914" rpy="0.0 0.0 ${0.25 * pi}" /--> <!-- MiR 250 Rviz-->
+      <origin xyz="0.3164 0.2064 0.1914" rpy="0.0 0.0 ${0.25 * pi}" /> <!-- MiR 250 CAD-->
+      <!--origin xyz="0.4288 0.2358 0.1914" rpy="0.0 0.0 ${0.25 * pi}" /-->  <!-- from visually matching up the meshes of the MiR and the laser scanner -->
+    </joint>
+    <xacro:sick_s300 prefix="${prefix}" link="front_laser_link" topic="f_scan" />
+    <joint name="${prefix}base_link_to_back_laser_joint" type="fixed">
+      <parent link="${prefix}base_link" />
+      <child link="${prefix}back_laser_link" />
+      <!--origin xyz="-0.2764 -0.2064 0.1914" rpy="0.0 0.0 ${-0.75 * pi}" /--> <!-- MiR 250 Rviz-->
+      <origin xyz="-0.3164 -0.2064 0.1914" rpy="0.0 0.0 ${-0.75 * pi}" /> <!-- MiR 250 CAD-->
+      <!--origin xyz="-0.3548 -0.2352 0.1914" rpy="0.0 0.0 ${-0.75 * pi}" /-->  <!-- from visually matching up the meshes of the MiR and the laser scanner -->
+    </joint>
+    <xacro:sick_s300 prefix="${prefix}" link="back_laser_link" topic="b_scan" />
+    <!-- Ultrasound sensors -->
+    <joint name="${prefix}us_1_joint" type="fixed">   <!-- right ultrasound -->
+      <parent link="${prefix}base_link" />
+      <child link="${prefix}us_1_frame" />
+      <origin xyz="0.45 -0.12 0.16 " rpy="0 0 0" />  <!-- from visually matching to the mesh of the MiR -->
+    </joint>
+    <link name="${prefix}us_1_frame" />
+    <joint name="${prefix}us_2_joint" type="fixed">   <!-- left ultrasound -->
+      <parent link="${prefix}base_link" />
+      <child link="${prefix}us_2_frame" />
+      <origin xyz="0.45 0.12 0.16 " rpy="0 0 0" />  <!-- from visually matching to the mesh of the MiR -->
+    </joint>
+    <link name="${prefix}us_2_frame" />
+    <!-- wheels -->
+    <xacro:actuated_wheel prefix="${prefix}" locationprefix="left" locationright="-1"/>
+    <xacro:actuated_wheel prefix="${prefix}" locationprefix="right" locationright="1"/>
+    <xacro:caster_wheel prefix="${prefix}" ns="${ns}" locationprefix="fl" locationright="-1" wheel_base_dx="${mir_100_front_caster_wheel_base_dx}"/>
+    <xacro:caster_wheel prefix="${prefix}" ns="${ns}" locationprefix="fr" locationright="1" wheel_base_dx="${mir_100_front_caster_wheel_base_dx}"/>
+    <xacro:caster_wheel prefix="${prefix}" ns="${ns}" locationprefix="bl" locationright="-1" wheel_base_dx="${mir_100_back_caster_wheel_base_dx}"/>
+    <xacro:caster_wheel prefix="${prefix}" ns="${ns}" locationprefix="br" locationright="1" wheel_base_dx="${mir_100_back_caster_wheel_base_dx}"/>
+    <joint name="${prefix}base_link_surface_joint" type="fixed">
+      <origin xyz="${mir_100_act_wheel_dx} 0 0.352" rpy="0 0 0" />
+      <parent link="${prefix}base_link" />
+      <child link="${prefix}surface" />
+      <axis xyz="0 0 1" />
+    </joint>
+    <link name="${prefix}surface"/>
+    <xacro:mir_100_wheel_transmissions prefix="${prefix}"/>
+    <xacro:p3d_base_controller prefix="${prefix}"/>
   </xacro:macro>
 </robot>

File: mir_description/urdf/include/sick_s300.urdf.xacro (robot description, xacro)
@@ -5,5 +5,5 @@
   <xacro:property name="laser_y" value="0.155" />
   <xacro:property name="laser_z" value="0.185" />
-  <xacro:property name="laser_mass" value="1.2" />
+  <xacro:property name="laser_mass" value="2.0" />
   <xacro:macro name="sick_s300" params="link topic prefix">
     <link name="${prefix}${link}">
@@ -30,5 +30,4 @@
       <material value="Gazebo/FlatBlack" />
       <sensor type="ray" name="${prefix}${link}">
-        <pose>0 0 0 0 0 0</pose>
         <visualize>false</visualize>
         <update_rate>12.5</update_rate>
@@ -49,5 +48,5 @@
           <noise>
             <type>gaussian</type>
-            <!-- Noise parameters based on published spec for S300 achieving
+              <!-- Noise parameters based on published spec for S300 achieving
                  "+-29mm" accuracy at range < 3m (~0.01 of the range) at
                  1 sigma. -->
@@ -56,7 +55,10 @@
           </noise>
         </ray>
-        <plugin name="gazebo_ros_${link}_controller" filename="libgazebo_ros_laser.so">
-          <frameName>${prefix}${link}</frameName>
-          <topicName>${topic}</topicName>
+        <plugin name="gazebo_ros_${link}_controller" filename="libgazebo_ros_ray_sensor.so">
+          <ros>
+            <remapping>~/out:=${prefix}${topic}</remapping>
+          </ros>
+          <output_type>sensor_msgs/LaserScan</output_type>
+          <frame_name>${prefix}${link}</frame_name>
         </plugin>
       </sensor>

File: mir_description/urdf/mir.urdf.xacro (robot description, xacro)
@@ -1,24 +1,23 @@
 <?xml version="1.0"?>
 <robot xmlns:xacro="http://ros.org/wiki/xacro"
-       name="mir" >
-  <!-- MiR base -->
-  <xacro:include filename="$(find mir_description)/urdf/include/mir_v1.urdf.xacro" />
+       name="mir_100" >
+  <!-- MiR100 base -->
+  <xacro:include filename="$(find mir_description)/urdf/include/mir_100_v1.urdf.xacro" />
   <xacro:include filename="$(find mir_description)/urdf/include/common.gazebo.xacro" />
+  <xacro:include filename="$(find mir_description)/urdf/include/mir_100.gazebo.xacro" />
   <xacro:arg name="tf_prefix" default="" />
-  <xacro:property name="tf_prefix_" value="$(arg tf_prefix)" />
-  <xacro:if value="${tf_prefix_ == ''}">
+  <!-- prefix can not start with a slash like a global namespace! results in TF errors -->
+  <xacro:property name="ns" value="$(arg tf_prefix)" />
+  <xacro:if value="${ns == ''}">
     <xacro:property name="prefix" value="" />
   </xacro:if>
-  <xacro:unless value="${tf_prefix_ == ''}">
-    <xacro:property name="prefix" value="${tf_prefix_}/" />
+  <xacro:unless value="${ns == ''}">
+    <xacro:property name="prefix" value="${ns}/" />
   </xacro:unless>
-  <xacro:mir prefix="${prefix}" />
-  <xacro:controller_plugin_gazebo robot_namespace=""/>
-  <!-- instead of the controller_plugin_gazebo, you can use the diffdrive controller like this:
-    <xacro:diff_controller_plugin_gazebo prefix=""
-      left_wheel_joint="left_wheel_joint"
-      right_wheel_joint="right_wheel_joint"
-      wheel_separation="${2*mir_act_wheel_dy}"
-      wheel_radius="${mir_act_wheel_radius}"/>
-  -->
+  <xacro:mir_100 prefix="${prefix}" ns="${ns}"/>
+  <xacro:diff_controller_plugin_gazebo prefix="${prefix}" ns="${ns}"
+    left_wheel_joint="${prefix}left_wheel_joint"
+    right_wheel_joint="${prefix}right_wheel_joint"
+    wheel_separation="${2*mir_100_act_wheel_dy}"
+    wheel_radius="${mir_100_act_wheel_radius}"/>
 </robot>
