Commit message: Removed unnecessary files

File: mir_description/urdf/include/mir_250_v1.urdf.xacro (robot description, xacro)
@@ -145,5 +145,5 @@
     </joint>
     <link name="${prefix}surface"/>
-    <joint name="${prefix}power_unit_joint" type="fixed">
+    <!-- <joint name="${prefix}power_unit_joint" type="fixed">
       <parent link="${prefix}base_link" />
       <child link="${prefix}power_unit" />
@@ -156,5 +156,4 @@
           <box size="0.73 0.56 0.4"/>
         </geometry>
-        <!-- Add material and other visual properties if needed -->
         <xacro:insert_block name="material_light_grey" />
       </visual>
@@ -164,7 +163,6 @@
           <box size="0.73 0.56 0.4"/>
        </geometry>
-        <!-- Add other collision properties if needed -->
       </collision>
-    </link>
+    </link> -->
     <!-- <xacro:arg name="name" default="ur"/> -->
     <!-- <xacro:arg name="ur_type" default="ur5e"/> -->
