Commit message: MiR250 with ros2_control

File: mir_description/urdf/include/caster.urdf.xacro (robot description, xacro)
@@ -80,5 +80,7 @@
         <origin xyz="0 0 0" rpy="${pi/2} 0 0" />
         <geometry>
-          <cylinder radius="${mir_100_caster_wheel_radius}" length="${mir_100_caster_wheel_width}" />
+          <!-- <cylinder radius="${mir_100_caster_wheel_radius}" length="${mir_100_caster_wheel_width}" /> -->
+          <cylinder radius="${mir_100_caster_wheel_radius}" length="0.00001" />
+          <!-- <sphere radius="${mir_100_caster_wheel_radius}" /> -->
         </geometry>
       </collision>
@@ -93,9 +95,14 @@
             <friction>
               <ode>
-                <mu>1.0</mu>
+                <!-- <mu>1.0</mu>
                 <mu2>1.0</mu2>
                 <fdir1>0 0 1</fdir1>
                 <slip1>0.0</slip1>
-                <slip2>0.5</slip2>
+                <slip2>0.5</slip2> -->
+                <mu>0.0</mu>
+                <mu2>0.0</mu2>
+                <fdir1>0 0 1</fdir1>
+                <slip1>0.0</slip1>
+                <slip2>0.0</slip2>
               </ode>
               <!-- <torsional>

File: mir_description/urdf/include/common.gazebo.xacro (robot description, xacro)
@@ -1,12 +1,14 @@
 <?xml version="1.0"?>
 <robot xmlns:xacro="http://ros.org/wiki/xacro">
-  <xacro:macro name="controller_plugin_gazebo" params="robot_namespace">
+  <xacro:macro name="controller_plugin_gazebo">   <!--params="robot_namespace">-->
     <gazebo>
       <plugin filename="libgazebo_ros2_control.so" name="gazebo_ros2_control">
+        <!--<parameters>/home/not_windows/Downloads/relffok_mir/src/mir_robot/mir_description/config/diffdrive_controller.yaml</parameters> -->
         <robot_param>robot_description</robot_param>
         <robot_param_node>robot_state_publisher</robot_param_node>
-        <xacro:unless value="${robot_namespace == ''}">
+        <parameters>$(find mir_description)/config/diffdrive_controller.yaml</parameters>
+        <!--<xacro:unless value="${robot_namespace == ''}">
           <robot_namespace>${robot_namespace}</robot_namespace>
-        </xacro:unless>
+        </xacro:unless>-->
         <control_period>0.001</control_period>
       </plugin>

File: mir_description/urdf/include/mir_100_v1.urdf.xacro (robot description, xacro)
@@ -8,4 +8,7 @@
   <xacro:include filename="$(find mir_description)/urdf/include/wheel.urdf.xacro" />
   <xacro:include filename="$(find mir_description)/urdf/include/caster.urdf.xacro" />
+  <!-- <xacro:include filename="$(find mir_description)/urdf/include/common.gazebo.xacro" /> -->
+  <!-- <xacro:include filename="$(find mir_description)/urdf/include/ros2_control.xacro" /> -->
+  <xacro:include filename="$(find ur_description)/urdf/ur_macro.xacro"/>
   <xacro:property name="deg_to_rad" value="0.017453293" />
   <!-- The inertia for the MiR platform is intentionally chosen to be smaller than
@@ -147,4 +150,108 @@
     <link name="${prefix}surface"/>
     <xacro:mir_100_wheel_transmissions prefix="${prefix}"/>
+    <joint name="${prefix}power_unit_joint" type="fixed">
+      <parent link="${prefix}base_link" />
+      <child link="${prefix}power_unit" />
+      <origin xyz="0 0 0.3" rpy="0 0 0" />
+    </joint>
+    <link name="${prefix}power_unit">
+      <visual>
+        <origin xyz="0 0 0.2" rpy="0 0 0" />
+        <geometry>
+          <box size="0.73 0.56 0.4"/>
+        </geometry>
+        <!-- Add material and other visual properties if needed -->
+        <xacro:insert_block name="material_light_grey" />
+      </visual>
+      <collision>
+        <origin xyz="0 0 0.2" rpy="0 0 0" />
+        <geometry>
+          <box size="0.73 0.56 0.4"/>
+       </geometry>
+        <!-- Add other collision properties if needed -->
+      </collision>
+    </link>
+    <!-- <xacro:arg name="name" default="ur"/> -->
+    <!-- <xacro:arg name="ur_type" default="ur5e"/> -->
+      <!-- parameters -->
+     <!-- <xacro:arg name="tf_prefix" default="" />
+     <xacro:arg name="joint_limit_params" default="$(find ur_description)/config/$(arg ur_type)/joint_limits.yaml"/>
+     <xacro:arg name="kinematics_params" default="$(find ur_description)/config/$(arg ur_type)/default_kinematics.yaml"/>
+     <xacro:arg name="physical_params" default="$(find ur_description)/config/$(arg ur_type)/physical_parameters.yaml"/>
+     <xacro:arg name="visual_params" default="$(find ur_description)/config/$(arg ur_type)/visual_parameters.yaml"/>
+     <xacro:arg name="transmission_hw_interface" default=""/>
+     <xacro:arg name="safety_limits" default="false"/>
+     <xacro:arg name="safety_pos_margin" default="0.15"/>
+     <xacro:arg name="safety_k_position" default="20"/> -->
+     <!-- ros2_control related parameters -->
+     <!-- <xacro:arg name="headless_mode" default="false" />
+     <xacro:arg name="robot_ip" default="0.0.0.0" />
+     <xacro:arg name="script_filename" default=""/>
+     <xacro:arg name="output_recipe_filename" default=""/>
+     <xacro:arg name="input_recipe_filename" default=""/>
+     <xacro:arg name="reverse_ip" default="0.0.0.0"/>
+     <xacro:arg name="script_command_port" default="50004"/>
+     <xacro:arg name="reverse_port" default="50001"/>
+     <xacro:arg name="script_sender_port" default="50002"/>
+     <xacro:arg name="trajectory_port" default="50003"/> -->
+     <!--   tool communication related parameters-->
+     <!-- <xacro:arg name="use_tool_communication" default="false" />
+     <xacro:arg name="tool_voltage" default="0" />
+     <xacro:arg name="tool_parity" default="0" />
+     <xacro:arg name="tool_baud_rate" default="115200" />
+     <xacro:arg name="tool_stop_bits" default="1" />
+     <xacro:arg name="tool_rx_idle_chars" default="1.5" />
+     <xacro:arg name="tool_tx_idle_chars" default="3.5" />
+     <xacro:arg name="tool_device_name" default="/tmp/ttyUR" />
+     <xacro:arg name="tool_tcp_port" default="54321" /> -->
+       <!-- Simulation parameters -->
+     <!-- <xacro:arg name="use_mock_hardware" default="false" />
+     <xacro:arg name="mock_sensor_commands" default="false" />
+     <xacro:arg name="sim_gazebo" default="true" />
+     <xacro:arg name="sim_ignition" default="false" />
+     <xacro:arg name="simulation_controllers" default="" /> -->
+     <!-- initial position for simulations (Mock Hardware, Gazebo, Ignition) -->
+     <!-- <xacro:arg name="initial_positions_file" default="$(find ur_description)/config/initial_positions.yaml"/> -->
+     <!-- convert to property to use substitution in function -->
+     <!-- <xacro:property name="initial_positions_file" default="$(arg initial_positions_file)"/>
+    <xacro:ur_robot
+     name="$(arg name)"
+     tf_prefix="ur"
+     parent="${prefix}base_link"
+     joint_limits_parameters_file="$(arg joint_limit_params)"
+     kinematics_parameters_file="$(arg kinematics_params)"
+     physical_parameters_file="$(arg physical_params)"
+     visual_parameters_file="$(arg visual_params)"
+     transmission_hw_interface="$(arg transmission_hw_interface)"
+     safety_limits="$(arg safety_limits)"
+     safety_pos_margin="$(arg safety_pos_margin)"
+     safety_k_position="$(arg safety_k_position)"
+     use_mock_hardware="$(arg use_mock_hardware)"
+     mock_sensor_commands="$(arg mock_sensor_commands)"
+     sim_gazebo="$(arg sim_gazebo)"
+     sim_ignition="$(arg sim_ignition)"
+     headless_mode="$(arg headless_mode)"
+     initial_positions="${xacro.load_yaml(initial_positions_file)}"
+     use_tool_communication="$(arg use_tool_communication)"
+     tool_voltage="$(arg tool_voltage)"
+     tool_parity="$(arg tool_parity)"
+     tool_baud_rate="$(arg tool_baud_rate)"
+     tool_stop_bits="$(arg tool_stop_bits)"
+     tool_rx_idle_chars="$(arg tool_rx_idle_chars)"
+     tool_tx_idle_chars="$(arg tool_tx_idle_chars)"
+     tool_device_name="$(arg tool_device_name)"
+     tool_tcp_port="$(arg tool_tcp_port)"
+     robot_ip="$(arg robot_ip)"
+     script_filename="$(arg script_filename)"
+     output_recipe_filename="$(arg output_recipe_filename)"
+     input_recipe_filename="$(arg input_recipe_filename)"
+     reverse_ip="$(arg reverse_ip)"
+     script_command_port="$(arg script_command_port)"
+     reverse_port="$(arg reverse_port)"
+     script_sender_port="$(arg script_sender_port)"
+     trajectory_port="$(arg trajectory_port)"
+     >
+     <origin xyz="0 0 0.7" rpy="0 0 0" />
+    </xacro:ur_robot> -->
     <xacro:p3d_base_controller prefix="${prefix}"/>
   </xacro:macro>

File: mir_description/urdf/include/wheel.urdf.xacro (robot description, xacro)
@@ -46,4 +46,7 @@
             <friction>
               <ode>
+                <!-- <mu>300.0</mu>
+                <mu2>300.0</mu2>
+                <fdir1>0 0 1</fdir1> -->
                 <mu>300.0</mu>
                 <mu2>300.0</mu2>

File: mir_description/urdf/mir.urdf.xacro (robot description, xacro)
@@ -4,6 +4,7 @@
   <!-- MiR100 base -->
   <xacro:include filename="$(find mir_description)/urdf/include/mir_100_v1.urdf.xacro" />
-  <xacro:include filename="$(find mir_description)/urdf/include/common.gazebo.xacro" />
-  <xacro:include filename="$(find mir_description)/urdf/include/mir_100.gazebo.xacro" />
+  <!-- <xacro:include filename="$(find mir_description)/urdf/include/common.gazebo.xacro" /> -->
+  <!-- <xacro:include filename="$(find mir_description)/urdf/include/mir_100.gazebo.xacro" /> -->
+  <!-- <xacro:include filename="$(find mir_description)/urdf/include/ros2_control.xacro" /> -->
   <xacro:arg name="tf_prefix" default="" />
   <!-- prefix can not start with a slash like a global namespace! results in TF errors -->
@@ -16,8 +17,38 @@
   </xacro:unless>
   <xacro:mir_100 prefix="${prefix}" ns="${ns}"/>
-  <xacro:diff_controller_plugin_gazebo prefix="${prefix}" ns="${ns}"
+  <!-- <xacro:diff_controller_plugin_gazebo prefix="${prefix}" ns="${ns}"
     left_wheel_joint="${prefix}left_wheel_joint"
     right_wheel_joint="${prefix}right_wheel_joint"
     wheel_separation="${2*mir_100_act_wheel_dy}"
-    wheel_radius="${mir_100_act_wheel_radius}"/>
+    wheel_radius="${mir_100_act_wheel_radius}"/> -->
+  <!-- <xacro:mir_ros2_control
+    left_wheel_joint="${prefix}left_wheel_joint"
+    right_wheel_joint="${prefix}right_wheel_joint"/>  -->
+  <ros2_control name="GazeboSystem" type="system">
+    <hardware>
+      <plugin>gazebo_ros2_control/GazeboSystem</plugin>
+    </hardware>
+    <joint name="left_wheel_joint">
+      <command_interface name="velocity">
+        <param name="min">-1</param>
+        <param name="max">1</param>
+      </command_interface>
+      <state_interface name="position"/>
+      <state_interface name="velocity"/>
+    </joint>
+    <joint name="right_wheel_joint">
+      <command_interface name="velocity">
+        <param name="min">-1</param>
+        <param name="max">1</param>
+      </command_interface>
+      <state_interface name="position"/>
+      <state_interface name="velocity"/>
+    </joint>
+  </ros2_control>
+  <gazebo>
+    <!-- Joint state publisher -->
+    <plugin filename="libgazebo_ros2_control.so" name="gazebo_ros2_control">
+      <parameters>$(find mir_description)/config/diffdrive_controller.yaml</parameters>
+    </plugin>
+  </gazebo>
 </robot>
