Commit message: Removed unnecessary files

File: mir_description/urdf/include/caster.urdf.xacro (robot description, xacro)
@@ -5,5 +5,5 @@
     <!-- caster hub -->
     <joint name="${prefix}${locationprefix}_caster_rotation_joint" type="continuous">
-      <origin xyz="${wheel_base_dx} ${-mir_100_caster_wheel_base_dy * locationright} ${mir_100_caster_wheel_base_dz}" rpy="0 0 0" />
+      <origin xyz="${wheel_base_dx} ${-mir_250_caster_wheel_base_dy * locationright} ${mir_250_caster_wheel_base_dz}" rpy="0 0 0" />
       <parent link="${prefix}base_link" />
       <child link="${prefix}${locationprefix}_caster_rotation_link" />
@@ -52,5 +52,5 @@
     <!-- caster wheel -->
     <joint name="${prefix}${locationprefix}_caster_wheel_joint" type="continuous">
-      <origin xyz="${mir_100_caster_wheel_dx} ${-mir_100_caster_wheel_dy * locationright} ${mir_100_caster_wheel_dz}" rpy="0 0 0" />
+      <origin xyz="${mir_250_caster_wheel_dx} ${-mir_250_caster_wheel_dy * locationright} ${mir_250_caster_wheel_dz}" rpy="0 0 0" />
       <parent link="${prefix}${locationprefix}_caster_rotation_link" />
       <child link="${prefix}${locationprefix}_caster_wheel_link" />
@@ -67,5 +67,5 @@
     </gazebo>
     <link name="${prefix}${locationprefix}_caster_wheel_link">
-      <xacro:cylinder_inertial mass="${mir_100_caster_wheel_mass}" radius="${mir_100_caster_wheel_radius}" length="${mir_100_caster_wheel_width}">
+      <xacro:cylinder_inertial mass="${mir_250_caster_wheel_mass}" radius="${mir_250_caster_wheel_radius}" length="${mir_250_caster_wheel_width}">
         <origin xyz="0 0 0" rpy="${0.5 * pi} 0 0" />
       </xacro:cylinder_inertial>
@@ -81,5 +81,5 @@
         <geometry>
           <!-- <cylinder radius="${mir_100_caster_wheel_radius}" length="${mir_100_caster_wheel_width}" /> -->
-          <cylinder radius="${mir_100_caster_wheel_radius}" length="0.00001" />
+          <cylinder radius="${mir_250_caster_wheel_radius}" length="0.00001" />
           <!-- <sphere radius="${mir_100_caster_wheel_radius}" /> -->
         </geometry>

File: mir_description/urdf/include/mir_250_v1.urdf.xacro (robot description, xacro)
@@ -3,11 +3,7 @@
   <xacro:include filename="$(find mir_description)/urdf/include/common_properties.urdf.xacro" />
   <xacro:include filename="$(find mir_description)/urdf/include/imu.gazebo.urdf.xacro" />
-  <xacro:include filename="$(find mir_description)/urdf/include/mir_100.gazebo.xacro" />
-  <xacro:include filename="$(find mir_description)/urdf/include/mir_100.transmission.xacro" />
   <xacro:include filename="$(find mir_description)/urdf/include/sick_s300.urdf.xacro" />
   <xacro:include filename="$(find mir_description)/urdf/include/wheel.urdf.xacro" />
   <xacro:include filename="$(find mir_description)/urdf/include/caster.urdf.xacro" />
-  <!-- <xacro:include filename="$(find mir_description)/urdf/include/common.gazebo.xacro" /> -->
-  <!-- <xacro:include filename="$(find mir_description)/urdf/include/ros2_control.xacro" /> -->
   <xacro:include filename="$(find ur_description)/urdf/ur_macro.xacro"/>
   <xacro:property name="deg_to_rad" value="0.017453293" />
@@ -21,24 +17,24 @@
   <xacro:property name="mir_base_inertial_y_length" value="0.30" />
   <xacro:property name="mir_base_inertial_z_length" value="0.20" />
-  <xacro:property name="mir_100_act_wheel_radius" value="0.100" />
-  <xacro:property name="mir_100_act_wheel_width" value="0.038" />
-  <xacro:property name="mir_100_act_wheel_mass" value="1.0" />
+  <xacro:property name="mir_250_act_wheel_radius" value="0.100" />
+  <xacro:property name="mir_250_act_wheel_width" value="0.038" />
+  <xacro:property name="mir_250_act_wheel_mass" value="1.0" />
   <!--xacro:property name="mir_100_act_wheel_dx" value="0.037646" /-->
-  <xacro:property name="mir_100_act_wheel_dx" value="-0.004485" />
+  <xacro:property name="mir_250_act_wheel_dx" value="-0.004485" />
   <!--xacro:property name="mir_100_act_wheel_dy" value="0.222604" /-->
-  <xacro:property name="mir_100_act_wheel_dy" value="0.2015" />
-  <xacro:property name="mir_100_caster_wheel_radius" value="0.0625" />
-  <xacro:property name="mir_100_caster_wheel_width" value="0.032" />
-  <xacro:property name="mir_100_caster_wheel_mass" value="1.0" />
-  <xacro:property name="mir_100_caster_wheel_dx" value="-0.0382" />
-  <xacro:property name="mir_100_caster_wheel_dy" value="0" />
-  <xacro:property name="mir_100_caster_wheel_dz" value="-0.094" />
+  <xacro:property name="mir_250_act_wheel_dy" value="0.2015" />
+  <xacro:property name="mir_250_caster_wheel_radius" value="0.0625" />
+  <xacro:property name="mir_250_caster_wheel_width" value="0.032" />
+  <xacro:property name="mir_250_caster_wheel_mass" value="1.0" />
+  <xacro:property name="mir_250_caster_wheel_dx" value="-0.0382" />
+  <xacro:property name="mir_250_caster_wheel_dy" value="0" />
+  <xacro:property name="mir_250_caster_wheel_dz" value="-0.094" />
   <!--xacro:property name="mir_100_front_caster_wheel_base_dx" value="0.341346" /-->
-  <xacro:property name="mir_100_front_caster_wheel_base_dx" value="0.3037" />
+  <xacro:property name="mir_250_front_caster_wheel_base_dx" value="0.3037" />
   <!--xacro:property name="mir_100_back_caster_wheel_base_dx" value="-0.270154" /-->
-  <xacro:property name="mir_100_back_caster_wheel_base_dx" value="-0.296" />
+  <xacro:property name="mir_250_back_caster_wheel_base_dx" value="-0.296" />
   <!--xacro:property name="mir_100_caster_wheel_base_dy" value="0.203" /-->
-  <xacro:property name="mir_100_caster_wheel_base_dy" value="0.188" />
-  <xacro:property name="mir_100_caster_wheel_base_dz" value="${mir_100_caster_wheel_radius - mir_100_caster_wheel_dz}" />
+  <xacro:property name="mir_250_caster_wheel_base_dy" value="0.188" />
+  <xacro:property name="mir_250_caster_wheel_base_dz" value="${mir_250_caster_wheel_radius - mir_250_caster_wheel_dz}" />
   <!-- MiR 100 complete mass 78.2kg (8.2kg battery) -->
   <!-- - 2x2kg sick laser = 4kg-->
@@ -46,7 +42,7 @@
   <!-- - 2x act wheels: 2kg -->
   <!--xacro:property name="mir_100_base_mass" value="66.96" /-->
-  <xacro:property name="mir_100_base_mass" value="97.0" />
+  <xacro:property name="mir_250_base_mass" value="97.0" />
   <xacro:property name="imu_stdev" value="0.00017" />
-  <xacro:macro name="mir_100" params="prefix ns">
+  <xacro:macro name="mir_250" params="prefix ns">
     <link name="${prefix}base_footprint" />
     <joint name="${prefix}base_joint" type="fixed">
@@ -56,9 +52,9 @@
     </joint>
     <link name="${prefix}base_link">
-      <xacro:box_inertial mass="${mir_100_base_mass}" x="${mir_base_inertial_x_length}" y="${mir_base_inertial_y_length}" z="${mir_base_inertial_z_length}">
-        <origin xyz="${mir_base_inertial_x + mir_100_act_wheel_dx} ${mir_base_inertial_y} ${mir_base_inertial_z}" rpy="0 0 0" />
+      <xacro:box_inertial mass="${mir_250_base_mass}" x="${mir_base_inertial_x_length}" y="${mir_base_inertial_y_length}" z="${mir_base_inertial_z_length}">
+        <origin xyz="${mir_base_inertial_x + mir_250_act_wheel_dx} ${mir_base_inertial_y} ${mir_base_inertial_z}" rpy="0 0 0" />
       </xacro:box_inertial>
       <visual>
-        <origin xyz="${mir_100_act_wheel_dx} 0 0" rpy="0 0 0" />
+        <origin xyz="${mir_250_act_wheel_dx} 0 0" rpy="0 0 0" />
         <geometry>
           <!--mesh filename="package://mir_description/meshes/visual/mir_100_base.stl" /-->
@@ -69,5 +65,5 @@
       </visual>
       <collision>
-        <origin xyz="${mir_100_act_wheel_dx} 0 0" rpy="0 0 0" />
+        <origin xyz="${mir_250_act_wheel_dx} 0 0" rpy="0 0 0" />
         <geometry>
           <!--mesh filename="package://mir_description/meshes/collision/mir_100_base.stl" /-->
@@ -138,10 +134,10 @@
     <xacro:actuated_wheel prefix="${prefix}" locationprefix="left" locationright="-1"/>
     <xacro:actuated_wheel prefix="${prefix}" locationprefix="right" locationright="1"/>
-    <xacro:caster_wheel prefix="${prefix}" ns="${ns}" locationprefix="fl" locationright="-1" wheel_base_dx="${mir_100_front_caster_wheel_base_dx}"/>
-    <xacro:caster_wheel prefix="${prefix}" ns="${ns}" locationprefix="fr" locationright="1" wheel_base_dx="${mir_100_front_caster_wheel_base_dx}"/>
-    <xacro:caster_wheel prefix="${prefix}" ns="${ns}" locationprefix="bl" locationright="-1" wheel_base_dx="${mir_100_back_caster_wheel_base_dx}"/>
-    <xacro:caster_wheel prefix="${prefix}" ns="${ns}" locationprefix="br" locationright="1" wheel_base_dx="${mir_100_back_caster_wheel_base_dx}"/>
+    <xacro:caster_wheel prefix="${prefix}" ns="${ns}" locationprefix="fl" locationright="-1" wheel_base_dx="${mir_250_front_caster_wheel_base_dx}"/>
+    <xacro:caster_wheel prefix="${prefix}" ns="${ns}" locationprefix="fr" locationright="1" wheel_base_dx="${mir_250_front_caster_wheel_base_dx}"/>
+    <xacro:caster_wheel prefix="${prefix}" ns="${ns}" locationprefix="bl" locationright="-1" wheel_base_dx="${mir_250_back_caster_wheel_base_dx}"/>
+    <xacro:caster_wheel prefix="${prefix}" ns="${ns}" locationprefix="br" locationright="1" wheel_base_dx="${mir_250_back_caster_wheel_base_dx}"/>
     <joint name="${prefix}base_link_surface_joint" type="fixed">
-      <origin xyz="${mir_100_act_wheel_dx} 0 0.352" rpy="0 0 0" />
+      <origin xyz="${mir_250_act_wheel_dx} 0 0.352" rpy="0 0 0" />
       <parent link="${prefix}base_link" />
       <child link="${prefix}surface" />
@@ -149,5 +145,4 @@
     </joint>
     <link name="${prefix}surface"/>
-    <xacro:mir_100_wheel_transmissions prefix="${prefix}"/>
     <joint name="${prefix}power_unit_joint" type="fixed">
       <parent link="${prefix}base_link" />
@@ -254,5 +249,4 @@
      <origin xyz="0 0 0.7" rpy="0 0 0" />
     </xacro:ur_robot> -->
-    <xacro:p3d_base_controller prefix="${prefix}"/>
   </xacro:macro>
 </robot>

File: mir_description/urdf/include/sick_s300.urdf.xacro (robot description, xacro)
@@ -30,5 +30,5 @@
       <material value="Gazebo/FlatBlack" />
       <sensor type="ray" name="${prefix}${link}">
-        <visualize>true</visualize>
+        <visualize>false</visualize>
         <update_rate>12.5</update_rate>
         <ray>

File: mir_description/urdf/include/wheel.urdf.xacro (robot description, xacro)
@@ -4,9 +4,9 @@
   <xacro:macro name="actuated_wheel" params="prefix  locationprefix locationright">
     <joint name="${prefix}${locationprefix}_wheel_joint" type="continuous">
-      <origin xyz="0.0 ${-mir_100_act_wheel_dy * locationright} ${mir_100_act_wheel_radius}" rpy="0 0 0" />
+      <origin xyz="0.0 ${-mir_250_act_wheel_dy * locationright} ${mir_250_act_wheel_radius}" rpy="0 0 0" />
       <parent link="${prefix}base_link" />
       <child link="${prefix}${locationprefix}_wheel_link" />
       <axis xyz="0 1 0" />
-      <limit effort="100" velocity="20.0" />
+      <limit effort="250" velocity="20.0" />
       <!-- <dynamics damping="0.0" friction="0.0"/> -->
       <!-- <gazebo reference="${prefix}${locationprefix}_wheel_joint">
@@ -15,5 +15,5 @@
     </joint>
     <link name="${prefix}${locationprefix}_wheel_link">
-      <xacro:cylinder_inertial mass="${mir_100_act_wheel_mass}" radius="${mir_100_act_wheel_radius}" length="${mir_100_act_wheel_width}">
+      <xacro:cylinder_inertial mass="${mir_250_act_wheel_mass}" radius="${mir_250_act_wheel_radius}" length="${mir_250_act_wheel_width}">
         <origin xyz="0 0 0" rpy="${0.5 * pi} 0 0" />
       </xacro:cylinder_inertial>
@@ -23,5 +23,5 @@
         <geometry>
           <!--mesh filename="package://mir_description/meshes/visual/wheel.stl" /-->
-          <cylinder radius="${mir_100_act_wheel_radius}" length="${mir_100_act_wheel_width}" />
+          <cylinder radius="${mir_250_act_wheel_radius}" length="${mir_250_act_wheel_width}" />
         </geometry>
         <xacro:insert_block name="material_dark_grey" />
@@ -30,5 +30,5 @@
         <origin xyz="0 0 0" rpy="${pi/2} 0 0" />
         <geometry>
-          <cylinder radius="${mir_100_act_wheel_radius}" length="${mir_100_act_wheel_width}" />
+          <cylinder radius="${mir_250_act_wheel_radius}" length="${mir_250_act_wheel_width}" />
         </geometry>
       </collision>
@@ -58,5 +58,5 @@
                 <coefficient>300</coefficient>
                 <use_patch_radius>false</use_patch_radius>
-                <surface_radius>${mir_100_act_wheel_radius}</surface_radius>
+                <surface_radius>${mir_250_act_wheel_radius}</surface_radius>
               </torsional>
             </friction>

File: mir_description/urdf/mir.urdf.xacro (robot description, xacro)
@@ -1,10 +1,7 @@
 <?xml version="1.0"?>
 <robot xmlns:xacro="http://ros.org/wiki/xacro"
-       name="mir_100" >
-  <!-- MiR100 base -->
-  <xacro:include filename="$(find mir_description)/urdf/include/mir_100_v1.urdf.xacro" />
-  <!-- <xacro:include filename="$(find mir_description)/urdf/include/common.gazebo.xacro" /> -->
-  <!-- <xacro:include filename="$(find mir_description)/urdf/include/mir_100.gazebo.xacro" /> -->
-  <!-- <xacro:include filename="$(find mir_description)/urdf/include/ros2_control.xacro" /> -->
+       name="mir_250" >
+  <!-- MiR250 base -->
+  <xacro:include filename="$(find mir_description)/urdf/include/mir_250_v1.urdf.xacro" />
   <xacro:arg name="tf_prefix" default="" />
   <!-- prefix can not start with a slash like a global namespace! results in TF errors -->
@@ -16,5 +13,5 @@
     <xacro:property name="prefix" value="${ns}/" />
   </xacro:unless>
-  <xacro:mir_100 prefix="${prefix}" ns="${ns}"/>
+  <xacro:mir_250 prefix="${prefix}" ns="${ns}"/>
   <!-- <xacro:diff_controller_plugin_gazebo prefix="${prefix}" ns="${ns}"
     left_wheel_joint="${prefix}left_wheel_joint"

Commit message: made changes to urdf and launch to get ign-gazebo running, check caster plugins

File: mir_description/urdf/include/caster.urdf.xacro (robot description, xacro)
@@ -36,5 +36,5 @@
         <origin xyz="0 0 0" rpy="0 0 0" />
         <geometry>
-          <mesh filename="package://mir_description/meshes/visual/caster_wheel_base.stl" />
+          <mesh filename="file://mir_description/meshes/visual/caster_wheel_base.stl" />
         </geometry>
         <xacro:insert_block name="material_silver" />
@@ -43,5 +43,5 @@
         <origin xyz="0 0 0" rpy="0 0 0" />
         <geometry>
-          <mesh filename="package://mir_description/meshes/collision/caster_wheel_base.stl" />
+          <mesh filename="file://mir_description/meshes/collision/caster_wheel_base.stl" />
         </geometry>
       </collision>
@@ -58,5 +58,6 @@
     </joint>
     <gazebo>
-      <plugin name="${locationprefix}_caster_wheel_joint_states" filename="libgazebo_ros_joint_state_publisher.so">
+      <!-- <plugin name="${locationprefix}_caster_wheel_joint_states" filename="libgazebo_ros_joint_state_publisher.so"> -->
+      <plugin name="${locationprefix}_caster_wheel_joint_states" filename="libignition-gazebo-joint-state-publisher.so"> <!-- Doesn't exist-->
         <ros>
           <namespace>${ns}</namespace>
@@ -73,5 +74,5 @@
         <origin xyz="0 0 0" rpy="0 0 0" />
         <geometry>
-          <mesh filename="package://mir_description/meshes/visual/wheel.stl" />
+          <mesh filename="file://mir_description/meshes/visual/wheel.stl" />
         </geometry>
         <xacro:insert_block name="material_dark_grey" />

File: mir_description/urdf/include/imu.gazebo.urdf.xacro (robot description, xacro)
@@ -71,5 +71,6 @@
           </linear_acceleration>
         </imu>
-        <plugin filename="libgazebo_ros_imu_sensor.so" name="imu_plugin">
+        <!-- <plugin filename="libgazebo_ros_imu_sensor.so" name="imu_plugin"> -->
+        <plugin filename="libignition-gazebo-imu-system.so" name="imu_plugin">
         <initial_orientation_as_reference>false</initial_orientation_as_reference>
           <ros>

File: mir_description/urdf/include/mir_250_v1.urdf.xacro (robot description, xacro)
@@ -59,5 +59,5 @@
         <geometry>
           <!--mesh filename="package://mir_description/meshes/visual/mir_100_base.stl" /-->
-          <mesh filename="package://mir_description/meshes/visual/mir_250_base.stl" />
+          <mesh filename="file://mir_description/meshes/visual/mir_250_base.stl" />
         </geometry>
         <!--xacro:insert_block name="material_white" /-->
@@ -67,6 +67,6 @@
         <origin xyz="${mir_250_act_wheel_dx} 0 0" rpy="0 0 0" />
         <geometry>
-          <!--mesh filename="package://mir_description/meshes/collision/mir_100_base.stl" /-->
-          <mesh filename="package://mir_description/meshes/collision/mir_250_base.stl" />
+          <!--mesh filename="file://mir_description/meshes/collision/mir_100_base.stl" /-->
+          <mesh filename="file://mir_description/meshes/collision/mir_250_base.stl" />
         </geometry>
       </collision>

File: mir_description/urdf/include/sick_s300.urdf.xacro (robot description, xacro)
@@ -11,5 +11,5 @@
         <origin xyz="0.0 0.0 0.0" rpy="${pi} 0 0" />
         <geometry>
-          <mesh filename="package://mir_description/meshes/visual/sick_lms-100.stl" />
+          <mesh filename="file://mir_description/meshes/visual/sick_lms-100.stl" />
         </geometry>
         <!-- <xacro:insert_block name="material_yellow" /> -->
@@ -19,5 +19,5 @@
         <origin xyz="0.0 0.0 0.0" rpy="${pi} 0 0" />
         <geometry>
-          <mesh filename="package://mir_description/meshes/visual/sick_lms-100.stl" />
+          <mesh filename="file://mir_description/meshes/visual/sick_lms-100.stl" />
         </geometry>
       </collision>
@@ -55,5 +55,7 @@
           </noise>
         </ray>
-        <plugin name="gazebo_ros_${link}_controller" filename="libgazebo_ros_ray_sensor.so">
+        <!-- <plugin name="gazebo_ros_${link}_controller" filename="libgazebo_ros_ray_sensor.so">     -->
+        <plugin name="gazebo_ros_${link}_controller" filename="libignition-gazebo-sensor-system.so">
+        <!-- Doesn't exist-->
           <ros>
             <remapping>~/out:=${prefix}${topic}</remapping>

File: mir_description/urdf/include/wheel.urdf.xacro (robot description, xacro)
@@ -22,5 +22,5 @@
         <origin xyz="0 0 0" rpy="${pi/2} 0 0" />
         <geometry>
-          <!--mesh filename="package://mir_description/meshes/visual/wheel.stl" /-->
+          <!--mesh filename="file://mir_description/meshes/visual/wheel.stl" /-->
           <cylinder radius="${mir_250_act_wheel_radius}" length="${mir_250_act_wheel_width}" />
         </geometry>

File: mir_description/urdf/mir.urdf.xacro (robot description, xacro)
@@ -22,5 +22,5 @@
     left_wheel_joint="${prefix}left_wheel_joint"
     right_wheel_joint="${prefix}right_wheel_joint"/>  -->
-  <ros2_control name="GazeboSystem" type="system">
+  <!-- <ros2_control name="GazeboSystem" type="system">
     <hardware>
       <plugin>gazebo_ros2_control/GazeboSystem</plugin>
@@ -42,8 +42,34 @@
       <state_interface name="velocity"/>
     </joint>
+  </ros2_control> -->
+  <ros2_control name="IgnitionSystem" type="system">
+    <hardware>
+      <plugin>ign_ros2_control/IgnitionSystem</plugin>
+    </hardware>
+    <joint name="left_wheel_joint">
+      <command_interface name="velocity">
+        <param name="min">-1</param>
+        <param name="max">1</param>
+      </command_interface>
+      <state_interface name="position"/>
+      <state_interface name="velocity"/>
+    </joint>
+    <joint name="right_wheel_joint">
+      <command_interface name="velocity">
+        <param name="min">-1</param>
+        <param name="max">1</param>
+      </command_interface>
+      <state_interface name="position"/>
+      <state_interface name="velocity"/>
+    </joint>
   </ros2_control>
+  <!-- <gazebo>
+    <plugin filename="libgazebo_ros2_control.so" name="gazebo_ros2_control">
+      <parameters>$(find mir_description)/config/diffdrive_controller.yaml</parameters>
+    </plugin>
+  </gazebo> -->
   <gazebo>
     <!-- Joint state publisher -->
-    <plugin filename="libgazebo_ros2_control.so" name="gazebo_ros2_control">
+    <plugin filename="ign_ros2_control-system" name="ign_ros2_control::IgnitionROS2ControlPlugin">
       <parameters>$(find mir_description)/config/diffdrive_controller.yaml</parameters>
     </plugin>

Commit message: caster wheel movement improved

File: mir_description/urdf/include/caster.urdf.xacro (robot description, xacro)
@@ -9,7 +9,7 @@
       <child link="${prefix}${locationprefix}_caster_rotation_link" />
       <axis xyz="0 0 1" />
-      <dynamics damping="0.0" friction="0.5"/>
+      <dynamics damping="0.0" friction="0.0"/>
     </joint>
-    <gazebo>
+    <!-- <gazebo>
       <plugin name="${locationprefix}_caster_rotation_joint_states" filename="libgazebo_ros_joint_state_publisher.so">
         <ros>
@@ -19,5 +19,5 @@
         <joint_name>${prefix}${locationprefix}_caster_rotation_joint</joint_name>
       </plugin>
-    </gazebo>
+    </gazebo> -->
     <link name="${prefix}${locationprefix}_caster_rotation_link">
       <inertial>
@@ -100,9 +100,9 @@
                 <slip1>0.0</slip1>
                 <slip2>0.5</slip2> -->
-                <mu>0.0</mu>
-                <mu2>0.0</mu2>
+                <mu>1.0</mu>
+                <mu2>1.0</mu2>
                 <fdir1>0 0 1</fdir1>
                 <slip1>0.0</slip1>
-                <slip2>0.0</slip2>
+                <slip2>0.5</slip2>
               </ode>
               <!-- <torsional>

File: mir_description/urdf/mir.urdf.xacro (robot description, xacro)
@@ -42,4 +42,36 @@
       <state_interface name="velocity"/>
     </joint>
+    <joint name="fl_caster_rotation_joint">
+      <state_interface name="position"/>
+      <state_interface name="velocity"/>
+    </joint>
+    <joint name="fr_caster_rotation_joint">
+      <state_interface name="position"/>
+      <state_interface name="velocity"/>
+    </joint>
+    <joint name="bl_caster_rotation_joint">
+      <state_interface name="position"/>
+      <state_interface name="velocity"/>
+    </joint>
+    <joint name="br_caster_rotation_joint">
+      <state_interface name="position"/>
+      <state_interface name="velocity"/>
+    </joint>
+    <joint name="fl__caster_wheel_joint">
+      <state_interface name="position"/>
+      <state_interface name="velocity"/>
+    </joint>
+    <joint name="fr__caster_wheel_joint">
+      <state_interface name="position"/>
+      <state_interface name="velocity"/>
+    </joint>
+    <joint name="bl__caster_wheel_joint">
+      <state_interface name="position"/>
+      <state_interface name="velocity"/>
+    </joint>
+    <joint name="br__caster_wheel_joint">
+      <state_interface name="position"/>
+      <state_interface name="velocity"/>
+    </joint>
   </ros2_control>
   <gazebo>
