Commit message: caster wheel behaviour improved

File: mir_description/urdf/include/caster.urdf.xacro (robot description, xacro)
@@ -57,5 +57,5 @@
       <axis xyz="0 1 0" />
     </joint>
-    <gazebo>
+    <!-- <gazebo>
       <plugin name="${locationprefix}_caster_wheel_joint_states" filename="libgazebo_ros_joint_state_publisher.so">
         <ros>
@@ -65,5 +65,5 @@
         <joint_name>${prefix}${locationprefix}_caster_wheel_joint</joint_name>
       </plugin>
-    </gazebo>
+    </gazebo> -->
     <link name="${prefix}${locationprefix}_caster_wheel_link">
       <xacro:cylinder_inertial mass="${mir_250_caster_wheel_mass}" radius="${mir_250_caster_wheel_radius}" length="${mir_250_caster_wheel_width}">

File: mir_description/urdf/mir.urdf.xacro (robot description, xacro)
@@ -58,17 +58,17 @@
       <state_interface name="velocity"/>
     </joint>
-    <joint name="fl__caster_wheel_joint">
+    <joint name="fl_caster_wheel_joint">
       <state_interface name="position"/>
       <state_interface name="velocity"/>
     </joint>
-    <joint name="fr__caster_wheel_joint">
+    <joint name="fr_caster_wheel_joint">
       <state_interface name="position"/>
       <state_interface name="velocity"/>
     </joint>
-    <joint name="bl__caster_wheel_joint">
+    <joint name="bl_caster_wheel_joint">
       <state_interface name="position"/>
       <state_interface name="velocity"/>
     </joint>
-    <joint name="br__caster_wheel_joint">
+    <joint name="br_caster_wheel_joint">
       <state_interface name="position"/>
       <state_interface name="velocity"/>

Commit message: Revert "Merge branch 'origin/ign-gazebo' into 'main'"
This reverts merge request !1

File: mir_description/urdf/include/caster.urdf.xacro (robot description, xacro)
@@ -36,5 +36,5 @@
         <origin xyz="0 0 0" rpy="0 0 0" />
         <geometry>
-          <mesh filename="file://mir_description/meshes/visual/caster_wheel_base.stl" />
+          <mesh filename="package://mir_description/meshes/visual/caster_wheel_base.stl" />
         </geometry>
         <xacro:insert_block name="material_silver" />
@@ -43,5 +43,5 @@
         <origin xyz="0 0 0" rpy="0 0 0" />
         <geometry>
-          <mesh filename="file://mir_description/meshes/collision/caster_wheel_base.stl" />
+          <mesh filename="package://mir_description/meshes/collision/caster_wheel_base.stl" />
         </geometry>
       </collision>
@@ -57,12 +57,6 @@
       <axis xyz="0 1 0" />
     </joint>
-<<<<<<< HEAD
-    <gazebo>
-      <!-- <plugin name="${locationprefix}_caster_wheel_joint_states" filename="libgazebo_ros_joint_state_publisher.so"> -->
-      <plugin name="${locationprefix}_caster_wheel_joint_states" filename="libignition-gazebo-joint-state-publisher.so"> <!-- Doesn't exist-->
-=======
     <!-- <gazebo>
       <plugin name="${locationprefix}_caster_wheel_joint_states" filename="libgazebo_ros_joint_state_publisher.so">
->>>>>>> cc6594dd9c4011d677f497c240b0c0fbea744c64
         <ros>
           <namespace>${ns}</namespace>
@@ -79,5 +73,5 @@
         <origin xyz="0 0 0" rpy="0 0 0" />
         <geometry>
-          <mesh filename="file://mir_description/meshes/visual/wheel.stl" />
+          <mesh filename="package://mir_description/meshes/visual/wheel.stl" />
         </geometry>
         <xacro:insert_block name="material_dark_grey" />

File: mir_description/urdf/include/imu.gazebo.urdf.xacro (robot description, xacro)
@@ -71,6 +71,5 @@
           </linear_acceleration>
         </imu>
-        <!-- <plugin filename="libgazebo_ros_imu_sensor.so" name="imu_plugin"> -->
-        <plugin filename="libignition-gazebo-imu-system.so" name="imu_plugin">
+        <plugin filename="libgazebo_ros_imu_sensor.so" name="imu_plugin">
         <initial_orientation_as_reference>false</initial_orientation_as_reference>
           <ros>

File: mir_description/urdf/include/mir_250_v1.urdf.xacro (robot description, xacro)
@@ -59,5 +59,5 @@
         <geometry>
           <!--mesh filename="package://mir_description/meshes/visual/mir_100_base.stl" /-->
-          <mesh filename="file://mir_description/meshes/visual/mir_250_base.stl" />
+          <mesh filename="package://mir_description/meshes/visual/mir_250_base.stl" />
         </geometry>
         <!--xacro:insert_block name="material_white" /-->
@@ -67,6 +67,6 @@
         <origin xyz="${mir_250_act_wheel_dx} 0 0" rpy="0 0 0" />
         <geometry>
-          <!--mesh filename="file://mir_description/meshes/collision/mir_100_base.stl" /-->
-          <mesh filename="file://mir_description/meshes/collision/mir_250_base.stl" />
+          <!--mesh filename="package://mir_description/meshes/collision/mir_100_base.stl" /-->
+          <mesh filename="package://mir_description/meshes/collision/mir_250_base.stl" />
         </geometry>
       </collision>

File: mir_description/urdf/include/sick_s300.urdf.xacro (robot description, xacro)
@@ -11,5 +11,5 @@
         <origin xyz="0.0 0.0 0.0" rpy="${pi} 0 0" />
         <geometry>
-          <mesh filename="file://mir_description/meshes/visual/sick_lms-100.stl" />
+          <mesh filename="package://mir_description/meshes/visual/sick_lms-100.stl" />
         </geometry>
         <!-- <xacro:insert_block name="material_yellow" /> -->
@@ -19,5 +19,5 @@
         <origin xyz="0.0 0.0 0.0" rpy="${pi} 0 0" />
         <geometry>
-          <mesh filename="file://mir_description/meshes/visual/sick_lms-100.stl" />
+          <mesh filename="package://mir_description/meshes/visual/sick_lms-100.stl" />
         </geometry>
       </collision>
@@ -55,7 +55,5 @@
           </noise>
         </ray>
-        <!-- <plugin name="gazebo_ros_${link}_controller" filename="libgazebo_ros_ray_sensor.so">     -->
-        <plugin name="gazebo_ros_${link}_controller" filename="libignition-gazebo-sensor-system.so">
-        <!-- Doesn't exist-->
+        <plugin name="gazebo_ros_${link}_controller" filename="libgazebo_ros_ray_sensor.so">
           <ros>
             <remapping>~/out:=${prefix}${topic}</remapping>

File: mir_description/urdf/include/wheel.urdf.xacro (robot description, xacro)
@@ -22,5 +22,5 @@
         <origin xyz="0 0 0" rpy="${pi/2} 0 0" />
         <geometry>
-          <!--mesh filename="file://mir_description/meshes/visual/wheel.stl" /-->
+          <!--mesh filename="package://mir_description/meshes/visual/wheel.stl" /-->
           <cylinder radius="${mir_250_act_wheel_radius}" length="${mir_250_act_wheel_width}" />
         </geometry>

File: mir_description/urdf/mir.urdf.xacro (robot description, xacro)
@@ -22,5 +22,5 @@
     left_wheel_joint="${prefix}left_wheel_joint"
     right_wheel_joint="${prefix}right_wheel_joint"/>  -->
-  <!-- <ros2_control name="GazeboSystem" type="system">
+  <ros2_control name="GazeboSystem" type="system">
     <hardware>
       <plugin>gazebo_ros2_control/GazeboSystem</plugin>
@@ -42,24 +42,4 @@
       <state_interface name="velocity"/>
     </joint>
-<<<<<<< HEAD
-  </ros2_control> -->
-  <ros2_control name="IgnitionSystem" type="system">
-    <hardware>
-      <plugin>ign_ros2_control/IgnitionSystem</plugin>
-    </hardware>
-    <joint name="left_wheel_joint">
-      <command_interface name="velocity">
-        <param name="min">-1</param>
-        <param name="max">1</param>
-      </command_interface>
-      <state_interface name="position"/>
-      <state_interface name="velocity"/>
-    </joint>
-    <joint name="right_wheel_joint">
-      <command_interface name="velocity">
-        <param name="min">-1</param>
-        <param name="max">1</param>
-      </command_interface>
-=======
     <joint name="fl_caster_rotation_joint">
       <state_interface name="position"/>
@@ -91,17 +71,11 @@
     </joint>
     <joint name="br_caster_wheel_joint">
->>>>>>> cc6594dd9c4011d677f497c240b0c0fbea744c64
       <state_interface name="position"/>
       <state_interface name="velocity"/>
     </joint>
   </ros2_control>
-  <!-- <gazebo>
-    <plugin filename="libgazebo_ros2_control.so" name="gazebo_ros2_control">
-      <parameters>$(find mir_description)/config/diffdrive_controller.yaml</parameters>
-    </plugin>
-  </gazebo> -->
   <gazebo>
     <!-- Joint state publisher -->
-    <plugin filename="ign_ros2_control-system" name="ign_ros2_control::IgnitionROS2ControlPlugin">
+    <plugin filename="libgazebo_ros2_control.so" name="gazebo_ros2_control">
       <parameters>$(find mir_description)/config/diffdrive_controller.yaml</parameters>
     </plugin>

Commit message: Lidar working with sdf, ros2control working with urdf.xacro

File: mir_description/urdf/include/caster.urdf.xacro (robot description, xacro)
@@ -36,5 +36,5 @@
         <origin xyz="0 0 0" rpy="0 0 0" />
         <geometry>
-          <mesh filename="file://mir_description/meshes/visual/caster_wheel_base.stl" />
+          <mesh filename="package://mir_description/meshes/visual/caster_wheel_base.stl" />
         </geometry>
         <xacro:insert_block name="material_silver" />
@@ -43,5 +43,5 @@
         <origin xyz="0 0 0" rpy="0 0 0" />
         <geometry>
-          <mesh filename="file://mir_description/meshes/collision/caster_wheel_base.stl" />
+          <mesh filename="package://mir_description/meshes/collision/caster_wheel_base.stl" />
         </geometry>
       </collision>
@@ -57,12 +57,7 @@
       <axis xyz="0 1 0" />
     </joint>
-<<<<<<< HEAD
+<!--
     <gazebo>
-      <!-- <plugin name="${locationprefix}_caster_wheel_joint_states" filename="libgazebo_ros_joint_state_publisher.so"> -->
-      <plugin name="${locationprefix}_caster_wheel_joint_states" filename="libignition-gazebo-joint-state-publisher.so"> <!-- Doesn't exist-->
-=======
-    <!-- <gazebo>
-      <plugin name="${locationprefix}_caster_wheel_joint_states" filename="libgazebo_ros_joint_state_publisher.so">
->>>>>>> cc6594dd9c4011d677f497c240b0c0fbea744c64
+      <plugin name="${locationprefix}_caster_wheel_joint_states" filename="libignition-gazebo-joint-state-publisher.so">
         <ros>
           <namespace>${ns}</namespace>
@@ -79,5 +74,5 @@
         <origin xyz="0 0 0" rpy="0 0 0" />
         <geometry>
-          <mesh filename="file://mir_description/meshes/visual/wheel.stl" />
+          <mesh filename="package://mir_description/meshes/visual/wheel.stl" />
         </geometry>
         <xacro:insert_block name="material_dark_grey" />
@@ -101,9 +96,4 @@
             <friction>
               <ode>
-                <!-- <mu>1.0</mu>
-                <mu2>1.0</mu2>
-                <fdir1>0 0 1</fdir1>
-                <slip1>0.0</slip1>
-                <slip2>0.5</slip2> -->
                 <mu>1.0</mu>
                 <mu2>1.0</mu2>

File: mir_description/urdf/include/imu.gazebo.urdf.xacro (robot description, xacro)
@@ -17,4 +17,5 @@
         <update_rate>${update_rate}</update_rate>
         <visualize>true</visualize>
+        <topic>${imu_topic}</topic>
         <imu>
           <angular_velocity>
@@ -71,13 +72,12 @@
           </linear_acceleration>
         </imu>
-        <!-- <plugin filename="libgazebo_ros_imu_sensor.so" name="imu_plugin"> -->
-        <plugin filename="libignition-gazebo-imu-system.so" name="imu_plugin">
+        <!-- <plugin filename="libgazebo_ros_imu_sensor.so" name="imu_plugin">
         <initial_orientation_as_reference>false</initial_orientation_as_reference>
           <ros>
             <namespace>${imu_topic}</namespace>
             <remapping>~/out:=data</remapping>
-            <frame_name>${imu_frame}</frame_name>  <!-- from real MiR -->
+            <frame_name>${imu_frame}</frame_name>
           </ros>
-        </plugin>
+        </plugin> -->
       </sensor>
     </gazebo>

File: mir_description/urdf/include/mir_250_v1.urdf.xacro (robot description, xacro)
@@ -59,5 +59,5 @@
         <geometry>
           <!--mesh filename="package://mir_description/meshes/visual/mir_100_base.stl" /-->
-          <mesh filename="file://mir_description/meshes/visual/mir_250_base.stl" />
+          <mesh filename="package://mir_description/meshes/visual/mir_250_base.stl" />
         </geometry>
         <!--xacro:insert_block name="material_white" /-->
@@ -68,5 +68,5 @@
         <geometry>
           <!--mesh filename="file://mir_description/meshes/collision/mir_100_base.stl" /-->
-          <mesh filename="file://mir_description/meshes/collision/mir_250_base.stl" />
+          <mesh filename="package://mir_description/meshes/collision/mir_250_base.stl" />
         </geometry>
       </collision>

File: mir_description/urdf/include/sick_s300.urdf.xacro (robot description, xacro)
@@ -11,5 +11,5 @@
         <origin xyz="0.0 0.0 0.0" rpy="${pi} 0 0" />
         <geometry>
-          <mesh filename="file://mir_description/meshes/visual/sick_lms-100.stl" />
+          <mesh filename="package://mir_description/meshes/visual/sick_lms-100.stl" />
         </geometry>
         <!-- <xacro:insert_block name="material_yellow" /> -->
@@ -19,5 +19,5 @@
         <origin xyz="0.0 0.0 0.0" rpy="${pi} 0 0" />
         <geometry>
-          <mesh filename="file://mir_description/meshes/visual/sick_lms-100.stl" />
+          <mesh filename="package://mir_description/meshes/visual/sick_lms-100.stl" />
         </geometry>
       </collision>
@@ -28,6 +28,6 @@
     <gazebo reference="${prefix}${link}">
       <!-- <material value="Gazebo/Yellow" /> -->
-      <material value="Gazebo/FlatBlack" />
-      <sensor type="ray" name="${prefix}${link}">
+      <!-- <material value="Gazebo/FlatBlack" /> -->
+      <!-- <sensor type="ray" name="${prefix}${link}">
         <visualize>false</visualize>
         <update_rate>12.5</update_rate>
@@ -36,5 +36,5 @@
             <horizontal>
               <samples>541</samples>
-              <resolution>1</resolution>  <!-- has to be 1; actual resolution will be computed from number of samples + min_angle/max_angle -->
+              <resolution>1</resolution>
               <min_angle>-2.09438</min_angle>
               <max_angle>2.09438</max_angle>
@@ -48,14 +48,9 @@
           <noise>
             <type>gaussian</type>
-              <!-- Noise parameters based on published spec for S300 achieving
-                 "+-29mm" accuracy at range < 3m (~0.01 of the range) at
-                 1 sigma. -->
             <mean>0.0</mean>
             <stddev>0.01</stddev>
           </noise>
         </ray>
-        <!-- <plugin name="gazebo_ros_${link}_controller" filename="libgazebo_ros_ray_sensor.so">     -->
-        <plugin name="gazebo_ros_${link}_controller" filename="libignition-gazebo-sensor-system.so">
-        <!-- Doesn't exist-->
+        <plugin name="gazebo_ros_${link}_controller" filename="libgazebo_ros_ray_sensor.so">
           <ros>
             <remapping>~/out:=${prefix}${topic}</remapping>
@@ -64,6 +59,42 @@
           <frame_name>${prefix}${link}</frame_name>
         </plugin>
+      </sensor> -->
+    <!-- </gazebo> -->
+      <sensor name="${prefix}${link}" type='gpu_lidar'>"
+        <pose relative_to="${prefix}${link}">0 0 0 0 0 0</pose>
+        <topic>${prefix}${topic}</topic>
+        <update_rate>12.5</update_rate>
+        <ray>
+            <scan>
+                <horizontal>
+                    <samples>541</samples>
+                    <resolution>1</resolution>
+                    <min_angle>-2.09438</min_angle>
+                    <max_angle>2.09438</max_angle>
+                </horizontal>
+                <!-- <vertical>
+                    <samples>1</samples>
+                    <resolution>0.01</resolution>
+                    <min_angle>0</min_angle>
+                    <max_angle>0</max_angle>
+                </vertical> -->
+            </scan>
+            <range>
+                <min>0.05</min>
+                <max>29.0</max>
+                <resolution>0.01</resolution>
+            </range>
+        </ray>
+        <always_on>true</always_on>
+        <visualize>true</visualize>
+        <gz_frame_id>${prefix}${link}</gz_frame_id>
       </sensor>
     </gazebo>
+    <!-- <gazebo>
+      <plugin filename="libignition-gazebo-sensors-system.so" name="ignition::gazebo::systems::Sensors">
+          <render_engine>ogre</render_engine>
+      </plugin>
+    </gazebo> -->
+    <!-- </link> -->
   </xacro:macro>
 </robot>

File: mir_description/urdf/mir.urdf.xacro (robot description, xacro)
@@ -42,5 +42,4 @@
       <state_interface name="velocity"/>
     </joint>
-<<<<<<< HEAD
   </ros2_control> -->
   <ros2_control name="IgnitionSystem" type="system">
@@ -61,5 +60,7 @@
         <param name="max">1</param>
       </command_interface>
-=======
+      <state_interface name="position"/>
+      <state_interface name="velocity"/>
+    </joint>
     <joint name="fl_caster_rotation_joint">
       <state_interface name="position"/>
@@ -91,5 +92,4 @@
     </joint>
     <joint name="br_caster_wheel_joint">
->>>>>>> cc6594dd9c4011d677f497c240b0c0fbea744c64
       <state_interface name="position"/>
       <state_interface name="velocity"/>
